File: PCB_files/easy-bee-counter-2026.kicad_pcb (KiCad board)
At the start: 2 copper layers, 346 x 40 mm, 82 parts, among them J1 Conn_01x04, Q1 IRLB8721PBF, Q2 IRLB8721PBF, U2 MCP23017_SP, U3 MCP23017_SP, U4 MCP23017_SP, U5 ESP32 C6 mini

Commit message: revised pcb design
Parts:
- removed H3, H6: MountingHole, MountingHole:MountingHole_3.2mm_M3
- added PD3: R_10k, Resistor_THT:R_Axial_DIN0207_L6.3mm_D2.5mm_P7.62mm_Horizontal, F.Cu at (124.4, 239.1)
- added Q3: IRLB8721PBF, Package_TO_SOT_THT:TO-220-3_Vertical, F.Cu at (138.2, 239.8)
- added R8: R_100, Resistor_THT:R_Axial_DIN0207_L6.3mm_D2.5mm_P7.62mm_Horizontal, F.Cu at (131.9, 235.4)
- R6, R7: value R_10k -> R_100
- RN7-22: renamed from RN7; value LED 1 -> LED 3
- moved RN3 36.3 mm to (218.5, 209.4)
- moved RN2-22 35.2 mm to (182.0, 209.4)
- moved Q2 11.5 mm to (138.2, 228.8)
- moved Q1 11.3 mm to (138.2, 217.8)
- moved PD1 9.28 mm to (124.4, 217.1)
- moved PD2 8.35 mm to (124.4, 228.1)
- moved R7 7.12 mm to (132.0, 224.5), turned to 180 degrees
- moved H1 7.06 mm to (112.9, 212.5)
- moved H2 6.28 mm to (241.8, 224.5)
- moved H5 5.05 mm to (429.2, 224.5)
- moved R6 3.54 mm to (132.0, 213.5), turned to 180 degrees
- moved R2 3.22 mm to (259.5, 222.1)
- moved C1 3.11 mm to (160.3, 218.6)
- moved C3 2.95 mm to (361.4, 217.8)
- moved R3 2.85 mm to (361.4, 221.7)
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- renumbered RN1 to RN1-100k1, RN2 to RN2-22, RN4 to RN4-22, RN5 to RN5-100k1, RN6 to RN6-100k1, RN8 to RN8-100k1, RN9 to RN9-100k1
Connections:
- Inner00 pad 1: /LED_BANK_1 -> +3.3V
- Inner01 pad 1: /LED_BANK_1 -> +3.3V
- Inner02 pad 1: /LED_BANK_1 -> +3.3V
- Inner03 pad 1: /LED_BANK_1 -> +3.3V
- Inner04 pad 1: /LED_BANK_1 -> +3.3V
- Inner05 pad 1: /LED_BANK_1 -> +3.3V
- Inner06 pad 1: /LED_BANK_1 -> +3.3V
- Inner07 pad 1: /LED_BANK_1 -> +3.3V
- Inner10 pad 1: /LED_BANK_1 -> +3.3V
- Inner11 pad 1: /LED_BANK_1 -> +3.3V
- Inner12 pad 1: /LED_BANK_1 -> +3.3V
- Inner13 pad 1: /LED_BANK_1 -> +3.3V
- Inner14 pad 1: /LED_BANK_2 -> +3.3V
- Inner15 pad 1: /LED_BANK_2 -> +3.3V
- Inner16 pad 1: /LED_BANK_2 -> +3.3V
- Inner17 pad 1: /LED_BANK_2 -> +3.3V
- Inner20 pad 1: /LED_BANK_2 -> +3.3V
- Inner21 pad 1: /LED_BANK_2 -> +3.3V
- Inner22 pad 1: /LED_BANK_2 -> +3.3V
- Inner23 pad 1: /LED_BANK_2 -> +3.3V
- Inner24 pad 1: /LED_BANK_2 -> +3.3V
- Inner25 pad 1: /LED_BANK_2 -> +3.3V
- Inner26 pad 1: /LED_BANK_2 -> +3.3V
- Inner27 pad 1: /LED_BANK_2 -> +3.3V
- J1 pad 3: /SDA -> /SDA_HiveScale
- J1 pad 4: /SDC -> /SCL_HiveScale
- Outer00 pad 1: /LED_BANK_1 -> +3.3V
- Outer01 pad 1: /LED_BANK_1 -> +3.3V
- Outer02 pad 1: /LED_BANK_1 -> +3.3V
- Outer03 pad 1: /LED_BANK_1 -> +3.3V
- Outer04 pad 1: /LED_BANK_1 -> +3.3V
- Outer05 pad 1: /LED_BANK_1 -> +3.3V
- Outer06 pad 1: /LED_BANK_1 -> +3.3V
- Outer07 pad 1: /LED_BANK_1 -> +3.3V
- Outer10 pad 1: /LED_BANK_1 -> +3.3V
- Outer11 pad 1: /LED_BANK_1 -> +3.3V
- Outer12 pad 1: /LED_BANK_1 -> +3.3V
- Outer13 pad 1: /LED_BANK_1 -> +3.3V
- Outer14 pad 1: /LED_BANK_2 -> +3.3V
- Outer15 pad 1: /LED_BANK_2 -> +3.3V
- Outer16 pad 1: /LED_BANK_2 -> +3.3V
- Outer17 pad 1: /LED_BANK_2 -> +3.3V
- Outer20 pad 1: /LED_BANK_2 -> +3.3V
- Outer21 pad 1: /LED_BANK_2 -> +3.3V
- Outer22 pad 1: /LED_BANK_2 -> +3.3V
- Outer23 pad 1: /LED_BANK_2 -> +3.3V
- Outer24 pad 1: /LED_BANK_2 -> +3.3V
- Outer25 pad 1: /LED_BANK_2 -> +3.3V
- Outer26 pad 1: /LED_BANK_2 -> +3.3V
- Outer27 pad 1: /LED_BANK_2 -> +3.3V
- RN2-22 pad 1: GND -> /LED_BANK_1
- RN4-22 pad 1: GND -> /LED_BANK_2
- RN7-22 pad 1: GND -> /LED_BANK_3
- U5 pad 11: unconnected-(U5-D10-Pad11) -> /GPIO6
- U5 pad 3: unconnected-(U5-D2-Pad3) -> /SDA_HiveScale
- U5 pad 4: unconnected-(U5-D3-Pad4) -> /SCL_HiveScale
Routing:
- net +3.3V: track 441.4 -> 892.7 mm, vias 1 -> 2
- net /LED_BANK_3: track 0.00 -> 267.6 mm, vias 0 -> 1
- net /LED_BANK_2: track 417.5 -> 155.9 mm, vias 0 -> 1
- net /LED_BANK_1: track 285.4 -> 46.2 mm
- net /GATE_04_IN: track 27.3 -> 87.8 mm
- net Net-(Inner24-K): track 34.1 -> 88.3 mm, vias 0 -> 2
- net Net-(Inner00-K): track 114.4 -> 66.3 mm
- net Net-(Inner26-K): track 51.3 -> 99.1 mm
- net Net-(Inner22-K): track 111.2 -> 64.2 mm
- net /GATE_00_OUT: track 141.4 -> 101.3 mm, vias 1 -> 2
- net Net-(Inner01-K): track 86.2 -> 46.2 mm, vias 1 -> 0
- net Net-(Inner21-K): track 83.2 -> 43.8 mm, vias 3 -> 0
- net Net-(Inner02-K): track 76.6 -> 39.3 mm
- net Net-(Inner03-K): track 75.6 -> 38.8 mm
- net /GATE_21_OUT: track 119.1 -> 82.5 mm, vias 1 -> 2
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Other:
- board text added: "3.3V GND SDA SCL"
- board text added: "BeeCounter2026-v0.2"
