File: PCB_files/easy-bee-counter-2026.kicad_pcb (KiCad board)
At the start: 2 copper layers, 346 x 40 mm, 83 parts, among them J1 Conn_01x04, Q1 IRLB8721PBF, Q2 IRLB8721PBF, Q3 IRLB8721PBF, U2 MCP23017_SP, U3 MCP23017_SP, U4 MCP23017_SP, U5 ESP32 C6 mini

Commit message: updated pcb design to v0.3
Connections:
- net /GPIO4 renamed /D8
- net /GPIO5 renamed /D9
- net /GPIO6 renamed /D10
Routing:
- net GND: vias 168 -> 177
Other:
- board text added: "BeeCounter2026-v0.3"
- board text removed: "BeeCounter2026-v0.2"
