File: PCB_files/easy-bee-counter-2026.kicad_sch (KiCad schematic)
At the start: 81 parts, among them J1 Conn_01x04, Q1 IRLB8721PBF, Q2 IRLB8721PBF, U2 MCP23017_SP, U3 MCP23017_SP, U4 MCP23017_SP, U5 ESP32 C6 mini

Commit message: revised pcb design
Parts:
- removed H3: MountingHole, MountingHole:MountingHole_3.2mm_M3, symbol Mechanical:MountingHole
- added PD3: R_10k, Resistor_THT:R_Axial_DIN0207_L6.3mm_D2.5mm_P7.62mm_Horizontal, symbol Device:R
- added Q3: IRLB8721PBF, Package_TO_SOT_THT:TO-220-3_Vertical, symbol Transistor_FET:IRLB8721PBF
- added R8: R_100, Resistor_THT:R_Axial_DIN0207_L6.3mm_D2.5mm_P7.62mm_Horizontal, symbol Device:R
- R6, R7: value R_10k -> R_100
- RN7-22: renamed from RN7; value LED 1 -> LED 3
- renumbered RN1 to RN1-100k1, RN2 to RN2-22, RN4 to RN4-22, RN5 to RN5-100k1, RN6 to RN6-100k1, RN8 to RN8-100k1, RN9 to RN9-100k1
Connections:
- net +3.3V: now also Inner00.1 (A), Inner01.1 (A), Inner02.1 (A), Inner03.1 (A), Inner04.1 (A), Inner05.1 (A), Inner06.1 (A), Inner07.1 (A), Inner10.1 (A), Inner11.1 (A), Inner12.1 (A), Inner13.1 (A), Inner14.1 (A), Inner15.1 (A), Inner16.1 (A), Inner17.1 (A), Inner20.1 (A), Inner21.1 (A), Inner22.1 (A), Inner23.1 (A), Inner24.1 (A), Inner25.1 (A), Inner26.1 (A), Inner27.1 (A), Outer00.1 (A), Outer01.1 (A), Outer02.1 (A), Outer03.1 (A), Outer04.1 (A), Outer05.1 (A), Outer06.1 (A), Outer07.1 (A), Outer10.1 (A), Outer11.1 (A), Outer12.1 (A), Outer13.1 (A), Outer14.1 (A), Outer15.1 (A), Outer16.1 (A), Outer17.1 (A), Outer20.1 (A), Outer21.1 (A), Outer22.1 (A), Outer23.1 (A), Outer24.1 (A), Outer25.1 (A), Outer26.1 (A), Outer27.1 (A)
- net GND: now also PD3.1, Q3.3 (S); no longer RN2-22.1 (common), RN4-22.1 (common), RN7-22.1 (common)
- net LED_BANK_1: now also RN2-22.1 (common); no longer Inner00.1 (A), Inner01.1 (A), Inner02.1 (A), Inner03.1 (A), Inner04.1 (A), Inner05.1 (A), Inner06.1 (A), Inner07.1 (A), Inner10.1 (A), Inner11.1 (A), Inner12.1 (A), Inner13.1 (A), Outer00.1 (A), Outer01.1 (A), Outer02.1 (A), Outer03.1 (A), Outer04.1 (A), Outer05.1 (A), Outer06.1 (A), Outer07.1 (A), Outer10.1 (A), Outer11.1 (A), Outer12.1 (A), Outer13.1 (A)
- net LED_BANK_2: now also RN4-22.1 (common); no longer Inner14.1 (A), Inner15.1 (A), Inner16.1 (A), Inner17.1 (A), Inner20.1 (A), Inner21.1 (A), Inner22.1 (A), Inner23.1 (A), Inner24.1 (A), Inner25.1 (A), Inner26.1 (A), Inner27.1 (A), Outer14.1 (A), Outer15.1 (A), Outer16.1 (A), Outer17.1 (A), Outer20.1 (A), Outer21.1 (A), Outer22.1 (A), Outer23.1 (A), Outer24.1 (A), Outer25.1 (A), Outer26.1 (A), Outer27.1 (A)
- net SDA: no longer J1.3 (Pin_3)
- net SDC: no longer J1.4 (Pin_4)
- net GPIO6: now reaches U5.11 (D10)
- net GPIO6: now also R8.2
- net SDA_HiveScale: now reaches U5.3 (D2)
- net SDA_HiveScale: now also J1.3 (Pin_3)
- net SCL_HiveScale: now reaches U5.4 (D3)
- net SCL_HiveScale: now also J1.4 (Pin_4)
- new net: PD3.2, Q3.1 (G), R8.1
- new net LED_BANK_3: Q3.2 (D), RN7-22.1 (common)
Other:
- moved on the sheet: H1, H2, H4, H5
