File: PCB_files/easy-bee-counter-2026.kicad_sch (KiCad schematic)
At the start: 83 parts, among them J1 Conn_01x04, Q1 IRLB8721PBF, Q2 IRLB8721PBF, Q3 IRLB8721PBF, U2 MCP23017_SP, U3 MCP23017_SP, U4 MCP23017_SP, U5 ESP32 C6 mini

Commit message: updated pcb design to v0.3
Connections:
- net GPIO4 renamed D8
- net GPIO5 renamed D9
- net GPIO6 renamed D10
Changed lines of the file:
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@@
 		)
 	)
-	(label "GPIO5"
+	(label "D9"
 		(at 80.01 208.28 0)
 		(effects
@@
 		)
 	)
-	(label "GPIO4"
+	(label "D8"
 		(at 48.26 73.66 270)
 		(effects
@@
 		)
 	)
-	(label "GPIO4"
+	(label "D8"
 		(at 80.01 205.74 0)
 		(effects
@@
 		)
 	)
-	(label "GPIO5"
+	(label "D9"
 		(at 49.53 99.06 270)
 		(effects
@@
 		)
 	)
-	(label "GPIO6"
+	(label "D10"
 		(at 49.53 127 270)
 		(effects
@@
 		)
 	)
-	(label "GPIO6"
+	(label "D10"
 		(at 80.01 210.82 0)
 		(effects
